File: reference-designs/asmr-module-backplane-x10-reference/asmr-module-backplane-x10-reference.kicad_pcb (KiCad board)
At the start: 2 copper layers, 380 x 67.5 mm, 45 parts, among them J1 PCI-36P, J10 PCI-36P, J2 PCI-36P, J3 PCI-36P, J4 PCI-36P, J5 PCI-36P, J6 PCI-36P, J7 PCI-36P, J8 PCI-36P, J9 PCI-36P

Commit message: Redesign backplane for 64 pin connector.
Parts:
- J1, J10, J2, J3, J4, J5, J6, J7, J8, J9: value PCI-36P -> PCI-64P; footprint CM_Connector_Edge:PCI-Slot-36-THD-FCI-10018783 -> CM_Connector_Edge:PCI-Slot-64-THD-FCI-10018784
- moved R14 7.52 mm to (146.3, 150.0)
- moved R13 7.52 mm to (145.1, 150.0)
- moved R11 6.58 mm to (141.4, 150.0)
- moved R12 6.58 mm to (142.6, 150.0)
- moved L1 1.20 mm to (122.0, 150.0), turned to -90 degrees
Connections:
- J1 pad A10: /CV -> +5V
- J1 pad A11: GNDS -> +5V
- J1 pad A13: /PATCH2 -> /COMA-SCK
- J1 pad A14: /PATCH4 -> /COMB-SCK
- J1 pad A15: /PATCH6 -> /CV
- J1 pad A16: /PATCH8 -> GNDS
- J1 pad A17: /PATCH10 -> /PATCH2
- J1 pad A18: /PATCH12 -> /PATCH4
- J1 pad A2: GND -> +18-24V
- J1 pad A3: +15V -> GND
- J1 pad A4: GND -> +15V
- J1 pad A5: -15V -> +15V
- J1 pad A7: +5V -> -15V
- J1 pad A8: /COMA-SCK -> -15V
- J1 pad A9: /COMB-SCK -> GND
- J1 pad B10: /GATE -> +5V
- J1 pad B11: GNDS -> +5V
- J1 pad B13: /PATCH1 -> /COMA-SDA
- J1 pad B14: /PATCH3 -> /COMB-SDA
- J1 pad B15: /PATCH5 -> /GATE
- J1 pad B16: /PATCH7 -> GNDS
- J1 pad B17: /PATCH9 -> /PATCH1
- J1 pad B18: /PATCH11 -> /PATCH3
- J1 pad B2: GND -> +18-24V
- J1 pad B3: +15V -> GND
- J1 pad B4: GND -> +15V
- J1 pad B5: -15V -> +15V
- J1 pad B7: +5V -> -15V
- J1 pad B8: /COMA-SDA -> -15V
- J1 pad B9: /COMB-SDA -> GND
- J10 pad A10: /CV -> +5V
- J10 pad A11: GNDS -> +5V
- J10 pad A13: /PATCH2 -> /COMA-SCK
- J10 pad A14: /PATCH4 -> /COMB-SCK
- J10 pad A15: /PATCH6 -> /CV
- J10 pad A16: /PATCH8 -> GNDS
- J10 pad A17: /PATCH10 -> /PATCH2
- J10 pad A18: /PATCH12 -> /PATCH4
- J10 pad A2: GND -> +18-24V
- J10 pad A3: +15V -> GND
- J10 pad A4: GND -> +15V
- J10 pad A5: -15V -> +15V
- J10 pad A7: +5V -> -15V
- J10 pad A8: /COMA-SCK -> -15V
- J10 pad A9: /COMB-SCK -> GND
- J10 pad B10: /GATE -> +5V
- J10 pad B11: GNDS -> +5V
- J10 pad B13: /PATCH1 -> /COMA-SDA
- J10 pad B14: /PATCH3 -> /COMB-SDA
- J10 pad B15: /PATCH5 -> /GATE
- J10 pad B16: /PATCH7 -> GNDS
- J10 pad B17: /PATCH9 -> /PATCH1
- J10 pad B18: /PATCH11 -> /PATCH3
- J10 pad B2: GND -> +18-24V
- J10 pad B3: +15V -> GND
- J10 pad B4: GND -> +15V
- J10 pad B5: -15V -> +15V
- J10 pad B7: +5V -> -15V
- J10 pad B8: /COMA-SDA -> -15V
- J10 pad B9: /COMB-SDA -> GND
- J2 pad A10: /CV -> +5V
- J2 pad A11: GNDS -> +5V
- J2 pad A13: /PATCH2 -> /COMA-SCK
- J2 pad A14: /PATCH4 -> /COMB-SCK
- J2 pad A15: /PATCH6 -> /CV
- J2 pad A16: /PATCH8 -> GNDS
- J2 pad A17: /PATCH10 -> /PATCH2
- J2 pad A18: /PATCH12 -> /PATCH4
- J2 pad A2: GND -> +18-24V
- J2 pad A3: +15V -> GND
- J2 pad A4: GND -> +15V
- J2 pad A5: -15V -> +15V
- J2 pad A7: +5V -> -15V
- J2 pad A8: /COMA-SCK -> -15V
- J2 pad A9: /COMB-SCK -> GND
- J2 pad B10: /GATE -> +5V
- J2 pad B11: GNDS -> +5V
- J2 pad B13: /PATCH1 -> /COMA-SDA
- J2 pad B14: /PATCH3 -> /COMB-SDA
- J2 pad B15: /PATCH5 -> /GATE
- J2 pad B16: /PATCH7 -> GNDS
- J2 pad B17: /PATCH9 -> /PATCH1
- J2 pad B18: /PATCH11 -> /PATCH3
- J2 pad B2: GND -> +18-24V
- J2 pad B3: +15V -> GND
- J2 pad B4: GND -> +15V
- J2 pad B5: -15V -> +15V
- J2 pad B7: +5V -> -15V
- J2 pad B8: /COMA-SDA -> -15V
- J2 pad B9: /COMB-SDA -> GND
- J3 pad A10: /CV -> +5V
- J3 pad A11: GNDS -> +5V
- J3 pad A13: /PATCH2 -> /COMA-SCK
- J3 pad A14: /PATCH4 -> /COMB-SCK
- J3 pad A15: /PATCH6 -> /CV
- J3 pad A16: /PATCH8 -> GNDS
- J3 pad A17: /PATCH10 -> /PATCH2
- J3 pad A18: /PATCH12 -> /PATCH4
- J3 pad A2: GND -> +18-24V
- J3 pad A3: +15V -> GND
- J3 pad A4: GND -> +15V
- J3 pad A5: -15V -> +15V
- J3 pad A7: +5V -> -15V
- J3 pad A8: /COMA-SCK -> -15V
- J3 pad A9: /COMB-SCK -> GND
- J3 pad B10: /GATE -> +5V
- J3 pad B11: GNDS -> +5V
- J3 pad B13: /PATCH1 -> /COMA-SDA
- J3 pad B14: /PATCH3 -> /COMB-SDA
- J3 pad B15: /PATCH5 -> /GATE
- J3 pad B16: /PATCH7 -> GNDS
- J3 pad B17: /PATCH9 -> /PATCH1
- J3 pad B18: /PATCH11 -> /PATCH3
- J3 pad B2: GND -> +18-24V
- J3 pad B3: +15V -> GND
- J3 pad B4: GND -> +15V
- J3 pad B5: -15V -> +15V
- J3 pad B7: +5V -> -15V
- J3 pad B8: /COMA-SDA -> -15V
- J3 pad B9: /COMB-SDA -> GND
- J4 pad A10: /CV -> +5V
- J4 pad A11: GNDS -> +5V
- J4 pad A13: /PATCH2 -> /COMA-SCK
- J4 pad A14: /PATCH4 -> /COMB-SCK
- J4 pad A15: /PATCH6 -> /CV
- J4 pad A16: /PATCH8 -> GNDS
- J4 pad A17: /PATCH10 -> /PATCH2
- J4 pad A18: /PATCH12 -> /PATCH4
- J4 pad A2: GND -> +18-24V
- J4 pad A3: +15V -> GND
- J4 pad A4: GND -> +15V
- J4 pad A5: -15V -> +15V
- J4 pad A7: +5V -> -15V
- J4 pad A8: /COMA-SCK -> -15V
- J4 pad A9: /COMB-SCK -> GND
- J4 pad B10: /GATE -> +5V
- J4 pad B11: GNDS -> +5V
- J4 pad B13: /PATCH1 -> /COMA-SDA
- J4 pad B14: /PATCH3 -> /COMB-SDA
- J4 pad B15: /PATCH5 -> /GATE
- J4 pad B16: /PATCH7 -> GNDS
- J4 pad B17: /PATCH9 -> /PATCH1
- J4 pad B18: /PATCH11 -> /PATCH3
- J4 pad B2: GND -> +18-24V
- J4 pad B3: +15V -> GND
- J4 pad B4: GND -> +15V
- J4 pad B5: -15V -> +15V
- J4 pad B7: +5V -> -15V
- J4 pad B8: /COMA-SDA -> -15V
- J4 pad B9: /COMB-SDA -> GND
- J5 pad A10: /CV -> +5V
- J5 pad A11: GNDS -> +5V
- J5 pad A13: /PATCH2 -> /COMA-SCK
- J5 pad A14: /PATCH4 -> /COMB-SCK
- J5 pad A15: /PATCH6 -> /CV
- J5 pad A16: /PATCH8 -> GNDS
- J5 pad A17: /PATCH10 -> /PATCH2
- J5 pad A18: /PATCH12 -> /PATCH4
- J5 pad A2: GND -> +18-24V
- J5 pad A3: +15V -> GND
- J5 pad A4: GND -> +15V
- J5 pad A5: -15V -> +15V
- J5 pad A7: +5V -> -15V
- J5 pad A8: /COMA-SCK -> -15V
- J5 pad A9: /COMB-SCK -> GND
- J5 pad B10: /GATE -> +5V
- J5 pad B11: GNDS -> +5V
- J5 pad B13: /PATCH1 -> /COMA-SDA
- J5 pad B14: /PATCH3 -> /COMB-SDA
- J5 pad B15: /PATCH5 -> /GATE
- J5 pad B16: /PATCH7 -> GNDS
- J5 pad B17: /PATCH9 -> /PATCH1
- J5 pad B18: /PATCH11 -> /PATCH3
- J5 pad B2: GND -> +18-24V
- J5 pad B3: +15V -> GND
- J5 pad B4: GND -> +15V
- J5 pad B5: -15V -> +15V
- J5 pad B7: +5V -> -15V
- J5 pad B8: /COMA-SDA -> -15V
- J5 pad B9: /COMB-SDA -> GND
- J6 pad A10: /CV -> +5V
- J6 pad A11: GNDS -> +5V
- J6 pad A13: /PATCH2 -> /COMA-SCK
- J6 pad A14: /PATCH4 -> /COMB-SCK
- J6 pad A15: /PATCH6 -> /CV
- J6 pad A16: /PATCH8 -> GNDS
- J6 pad A17: /PATCH10 -> /PATCH2
- J6 pad A18: /PATCH12 -> /PATCH4
- J6 pad A2: GND -> +18-24V
- J6 pad A3: +15V -> GND
- J6 pad A4: GND -> +15V
- J6 pad A5: -15V -> +15V
- J6 pad A7: +5V -> -15V
- J6 pad A8: /COMA-SCK -> -15V
- J6 pad A9: /COMB-SCK -> GND
- J6 pad B10: /GATE -> +5V
- J6 pad B11: GNDS -> +5V
- J6 pad B13: /PATCH1 -> /COMA-SDA
- J6 pad B14: /PATCH3 -> /COMB-SDA
- J6 pad B15: /PATCH5 -> /GATE
- J6 pad B16: /PATCH7 -> GNDS
- J6 pad B17: /PATCH9 -> /PATCH1
- J6 pad B18: /PATCH11 -> /PATCH3
- J6 pad B2: GND -> +18-24V
- J6 pad B3: +15V -> GND
- J6 pad B4: GND -> +15V
- J6 pad B5: -15V -> +15V
- J6 pad B7: +5V -> -15V
- J6 pad B8: /COMA-SDA -> -15V
- J6 pad B9: /COMB-SDA -> GND
- J7 pad A10: /CV -> +5V
- J7 pad A11: GNDS -> +5V
- J7 pad A13: /PATCH2 -> /COMA-SCK
- J7 pad A14: /PATCH4 -> /COMB-SCK
- J7 pad A15: /PATCH6 -> /CV
- J7 pad A16: /PATCH8 -> GNDS
- J7 pad A17: /PATCH10 -> /PATCH2
- J7 pad A18: /PATCH12 -> /PATCH4
- J7 pad A2: GND -> +18-24V
- J7 pad A3: +15V -> GND
- J7 pad A4: GND -> +15V
- J7 pad A5: -15V -> +15V
- J7 pad A7: +5V -> -15V
- J7 pad A8: /COMA-SCK -> -15V
- J7 pad A9: /COMB-SCK -> GND
- J7 pad B10: /GATE -> +5V
- J7 pad B11: GNDS -> +5V
- J7 pad B13: /PATCH1 -> /COMA-SDA
- J7 pad B14: /PATCH3 -> /COMB-SDA
- J7 pad B15: /PATCH5 -> /GATE
- J7 pad B16: /PATCH7 -> GNDS
- J7 pad B17: /PATCH9 -> /PATCH1
- J7 pad B18: /PATCH11 -> /PATCH3
- J7 pad B2: GND -> +18-24V
- J7 pad B3: +15V -> GND
- J7 pad B4: GND -> +15V
- J7 pad B5: -15V -> +15V
- J7 pad B7: +5V -> -15V
- J7 pad B8: /COMA-SDA -> -15V
- J7 pad B9: /COMB-SDA -> GND
- J8 pad A10: /CV -> +5V
- J8 pad A11: GNDS -> +5V
- J8 pad A13: /PATCH2 -> /COMA-SCK
- J8 pad A14: /PATCH4 -> /COMB-SCK
- J8 pad A15: /PATCH6 -> /CV
- J8 pad A16: /PATCH8 -> GNDS
- J8 pad A17: /PATCH10 -> /PATCH2
- J8 pad A18: /PATCH12 -> /PATCH4
- J8 pad A2: GND -> +18-24V
- J8 pad A3: +15V -> GND
- J8 pad A4: GND -> +15V
- J8 pad A5: -15V -> +15V
- J8 pad A7: +5V -> -15V
- J8 pad A8: /COMA-SCK -> -15V
- J8 pad A9: /COMB-SCK -> GND
- J8 pad B10: /GATE -> +5V
- J8 pad B11: GNDS -> +5V
- J8 pad B13: /PATCH1 -> /COMA-SDA
- J8 pad B14: /PATCH3 -> /COMB-SDA
- J8 pad B15: /PATCH5 -> /GATE
- J8 pad B16: /PATCH7 -> GNDS
- J8 pad B17: /PATCH9 -> /PATCH1
- J8 pad B18: /PATCH11 -> /PATCH3
- J8 pad B2: GND -> +18-24V
- J8 pad B3: +15V -> GND
- J8 pad B4: GND -> +15V
- J8 pad B5: -15V -> +15V
- J8 pad B7: +5V -> -15V
- J8 pad B8: /COMA-SDA -> -15V
- J8 pad B9: /COMB-SDA -> GND
- J9 pad A10: /CV -> +5V
- J9 pad A11: GNDS -> +5V
- J9 pad A13: /PATCH2 -> /COMA-SCK
- J9 pad A14: /PATCH4 -> /COMB-SCK
- J9 pad A15: /PATCH6 -> /CV
- J9 pad A16: /PATCH8 -> GNDS
- J9 pad A17: /PATCH10 -> /PATCH2
- J9 pad A18: /PATCH12 -> /PATCH4
- J9 pad A2: GND -> +18-24V
- J9 pad A3: +15V -> GND
- J9 pad A4: GND -> +15V
- J9 pad A5: -15V -> +15V
- J9 pad A7: +5V -> -15V
- J9 pad A8: /COMA-SCK -> -15V
- J9 pad A9: /COMB-SCK -> GND
- J9 pad B10: /GATE -> +5V
- J9 pad B11: GNDS -> +5V
- J9 pad B13: /PATCH1 -> /COMA-SDA
- J9 pad B14: /PATCH3 -> /COMB-SDA
- J9 pad B15: /PATCH5 -> /GATE
- J9 pad B16: /PATCH7 -> GNDS
- J9 pad B17: /PATCH9 -> /PATCH1
- J9 pad B18: /PATCH11 -> /PATCH3
- J9 pad B2: GND -> +18-24V
- J9 pad B3: +15V -> GND
- J9 pad B4: GND -> +15V
- J9 pad B5: -15V -> +15V
- J9 pad B7: +5V -> -15V
- J9 pad B8: /COMA-SDA -> -15V
- J9 pad B9: /COMB-SDA -> GND
Routing:
- net GNDS: track 0.21 -> 375.2 mm
- net /PATCH22: track 0.00 -> 369.3 mm
- net /PATCH27: track 0.00 -> 368.6 mm, vias 0 -> 9
- net /PATCH14: track 0.00 -> 368.6 mm
- net /PATCH26: track 0.00 -> 368.6 mm
- net /PATCH18: track 0.00 -> 368.5 mm
- net /PATCH23: track 0.00 -> 368.1 mm, vias 0 -> 9
- net /PATCH24: track 0.00 -> 368.1 mm, vias 0 -> 9
- net /PATCH19: track 0.00 -> 368.0 mm, vias 0 -> 9
- net /PATCH15: track 0.00 -> 368.0 mm, vias 0 -> 9
- net /PATCH31: track 0.00 -> 368.0 mm, vias 0 -> 9
- net /PATCH20: track 0.00 -> 367.9 mm, vias 0 -> 9
- net /PATCH28: track 0.00 -> 367.9 mm, vias 0 -> 9
- net /PATCH13: track 0.00 -> 367.7 mm
- net /PATCH16: track 0.00 -> 367.7 mm, vias 0 -> 9
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- removed copper zone on F.Cu, net GNDS
Other:
- board size 380 x 67.5 mm -> 385 x 67.5 mm
