File: reference-designs/asmr-dreamland-pcb/asmr-dreamland-pcb.kicad_pcb (KiCad board)
At the start: 2 copper layers, 136 x 72 mm, 23 parts, among them J10 Conn_01x10, J11 Conn_01x10, J12 Conn_01x10, J13 Conn_01x10, J14 Conn_01x03, J15 Conn_01x03, J16 Conn_01x03, J17 Conn_01x03, J18 Conn_01x08, J2 Conn_01x06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

Commit message: More changes to DreamLand.
Routing:
- net GND_CH: vias 98 -> 101
Other:
- outline, holes or cut-outs redrawn
- board text added: "HOLE"
Changed lines of the file:
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@@
+	)
+	(gr_rect
+		(start 109 54.5)
+		(end 191 109.5)
+		(stroke
+			(width 0.4)
+			(type default)
+		)
+		(fill no)
+		(layer "B.SilkS")
 	)
 	(gr_rect
@@
 		(layer "Edge.Cuts")
 	)
+	(gr_rect
+		(start 206 99)
+		(end 214 105)
+		(stroke
+			(width 0.05)
+			(type default)
+		)
+		(fill no)
+		(layer "Edge.Cuts")
+	)
+	(gr_rect
+		(start 87 98.5)
+		(end 95 102.5)
+		(stroke
+			(width 0.05)
+			(type default)
+		)
+		(fill no)
+		(layer "Edge.Cuts")
+	)
 	(gr_line
 		(start 105 115)
@@
 			(type default)
 		)
+		(layer "Edge.Cuts")
+	)
+	(gr_rect
+		(start 87 53)
+		(end 95 57)
+		(stroke
+			(width 0.05)
+			(type default)
+		)
+		(fill no)
+		(layer "Edge.Cuts")
+	)
+	(gr_rect
+		(start 206 54)
+		(end 214 60)
+		(stroke
+			(width 0.05)
+			(type default)
+		)
+		(fill no)
 		(layer "Edge.Cuts")
 	)
@@
 		)
 	)
+	(gr_text "HOLE"
+		(at 91 55 0)
+		(layer "Edge.Cuts")
+		(effects
+			(font
+				(size 1 1)
+				(thickness 0.15)
+			)
+		)
+	)
+	(gr_text "HOLE"
+		(at 210 102 0)
+		(layer "Edge.Cuts")
+		(effects
+			(font
+				(size 1 1)
+				(thickness 0.15)
+			)
+		)
+	)
+	(gr_text "HOLE"
+		(at 209.5 57 0)
+		(layer "Edge.Cuts")
+		(effects
+			(font
+				(size 1 1)
+				(thickness 0.15)
+			)
+		)
+	)
+	(gr_text "HOLE"
+		(at 90.5 100.5 0)
+		(layer "Edge.Cuts")
+		(effects
+			(font
+				(size 1 1)
+				(thickness 0.15)
+			)
+		)
+	)
 	(segment
 		(start 118.5 121)
@@
 	)
 	(via
-		(at 90 50)
-		(size 0.6)
-		(drill 0.3)
-		(layers "F.Cu" "B.Cu")
-		(free yes)
-		(net 18)
-	)
-	(via
 		(at 170 86)
 		(size 0.6)
@@
 	)
 	(via
+		(at 110 44)
+		(size 0.6)
+		(drill 0.3)
+		(layers "F.Cu" "B.Cu")
+		(free yes)
+		(net 18)
+	)
+	(via
 		(at 113.5 118.5)
 		(size 0.6)
@@
 	)
 	(via
+		(at 90 44)
+		(size 0.6)
+		(drill 0.3)
+		(layers "F.Cu" "B.Cu")
+		(free yes)
+		(net 18)
+	)
+	(via
 		(at 116.5 118.5)
 		(size 0.6)
@@
 	)
 	(via
+		(at 100 44)
+		(size 0.6)
+		(drill 0.3)
+		(layers "F.Cu" "B.Cu")
+		(free yes)
+		(net 18)
+	)
+	(via
 		(at 191 59)
 		(size 0.6)
@@
 		(size 0.6)
 		(drill 0.3)
+		(layers "F.Cu" "B.Cu")
+		(free yes)
+		(net 18)
+	)
+	(via
+		(at 130 44)
+		(size 0.6)
+		(drill 0.3)
