File: reference-designs/asmr-dreamland/asmr-dreamland-face-plate/asmr-dreamland-face-plate.kicad_pcb (KiCad board)
At the start: 2 copper layers, 40 x 159.8 mm, 0 parts

Commit message: Designed DreamLand face plate.
Routing:
- added copper zone on F.Cu, net (none)
Other:
- board size 40 x 159.8 mm -> 40 x 159.6 mm
- board text added: "1"
- board text added: "2"
- board text added: "3"
- board text added: "4"
- board text added: "A S M R"
- board text added: "DreamLand"
