File: reference-designs/asmr-dreamland/asmr-dreamland-face-plate/asmr-dreamland-face-plate.kicad_sch (KiCad schematic)
At the start: 0 parts

Commit message: Designed DreamLand face plate.
Other:
- title: Single Module Face Plate Reference Design -> DreamLand Module Face Plate
Changed lines of the file:
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@@
 	(paper "A4")
 	(title_block
-		(title "Single Module Face Plate Reference Design")
+		(title "DreamLand Module Face Plate")
 		(date "2025-08-12")
 		(rev "A")
 		(company "by Circuit Monkey")
-		(comment 1 "ASMR :: Advanced Synth Module Rack")
-		(comment 2 "Face Plate for a AMSR Single Slot Module")
+		(comment 1 "for ASMR :: Advanced Synth Module Rack")
+		(comment 2 "Face Plate for DreamLand Module")
 	)
 	(sheet_instances

Commit message: Final DreamLand faceplate?
Other:
- note added: "- Large Hole, 9mm. Pots on PCB, Model RV111. Tayda: A-5538 (or similar) - Med Hole, 8mm. LED Holder, for 5mm LED. Tayda: A-366 - Small Hole, 6mm. TRS Jack, 3.5mm. Tayda: A-2585, A-4338, A-4317"
- note added: "Notes:"
Changed lines of the file:
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@@
 		(comment 2 "Face Plate for DreamLand Module")
+	)
+	(text "Notes:"
+		(exclude_from_sim no)
+		(at 48.006 61.722 0)
+		(effects
+			(font
+				(size 3 3)
+				(thickness 0.6)
+				(bold yes)
+			)
+			(justify left bottom)
+		)
+	)
+	(text " - Large Hole, 9mm.  Pots on PCB, Model RV111. Tayda: A-5538 (or similar)\n - Med Hole, 8mm. LED Holder, for 5mm LED. Tayda: A-366\n - Small Hole, 6mm.  TRS Jack, 3.5mm.  Tayda: A-2585, A-4338, A-4317"
+		(exclude_from_sim no)
+		(at 52.07 63.5 0)
+		(effects
+			(font
+				(size 3 3)
+				(thickness 0.254)
+				(bold yes)
+			)
+			(justify left top)
+		)
 	)
 	(sheet_instances
