File: reference-designs/asmr-module-face-plate-reference/asmr-module-face-plate-reference.kicad_sch (KiCad schematic)
At the start: 0 parts

Commit message: Tune faceplate design.
Other:
- note added: "- Large Hole, 9mm. Pots on PCB, Model RV111. Tayda: A-5538 (or similar) - Med Hole, 8mm. LED Holder, for 5mm LED. Tayda: A-366 - Small Hole, 6mm. TRS Jack, 3.5mm. Tayda: A-2585, A-4338, A-4317"
- note added: "For your consideration:"
Changed lines of the file:
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@@
 		(comment 2 "Face Plate for a AMSR Single Slot Module")
+	)
+	(text " - Large Hole, 9mm.  Pots on PCB, Model RV111. Tayda: A-5538 (or similar)\n - Med Hole, 8mm. LED Holder, for 5mm LED. Tayda: A-366\n - Small Hole, 6mm.  TRS Jack, 3.5mm.  Tayda: A-2585, A-4338, A-4317"
+		(exclude_from_sim no)
+		(at 55.118 52.832 0)
+		(effects
+			(font
+				(size 3 3)
+				(thickness 0.254)
+				(bold yes)
+			)
+			(justify left top)
+		)
+	)
+	(text "For your consideration:"
+		(exclude_from_sim no)
+		(at 51.054 51.054 0)
+		(effects
+			(font
+				(size 3 3)
+				(thickness 0.6)
+				(bold yes)
+			)
+			(justify left bottom)
+		)
 	)
 	(sheet_instances
