File: modules/hagiwo-unison-vco/hagiwo-unison-vco.kicad_pcb (KiCad board)
At the start: 2 copper layers, 136 x 72 mm, 47 parts, among them J1 JST-SH, J2 JST-SH, J3 JST-SH, J4 Conn_01x02_MountingPin, U1 XIAO RA4M1, U2 TL074

Commit message: Updates to Unison board.
Parts:
- removed D1, D2, D3, D4: BAT43W-V, Diode_SMD:D_SOD-123
- added D5: D1213A, CM_Chip_Packages:SOT-25, F.Cu at (120.0, 74.9)
- moved C1 1.80 mm to (117.6, 75.0)
Routing:
- net GNDS: track 127.8 -> 120.2 mm
- net +3V3: track 195.1 -> 187.8 mm, vias 8 -> 7
- net V-OCT: track 36.1 -> 30.7 mm
- net OSC2_VOL: track 48.8 -> 46.1 mm
- net /OUT_TIP: track 53.1 -> 52.3 mm
- net Net-(R3-Pad1): track 16.8 -> 17.5 mm
- net SCL: track 17.3 -> 16.7 mm
- net -15V: track 42.6 -> 43.1 mm
- net GND_CH: vias 9 -> 127
