File: modules/hagiwo-unison-vco/hagiwo-unison-vco.kicad_sch (KiCad schematic)
At the start: 47 parts, among them J1 JST-SH, J2 JST-SH, J3 JST-SH, J4 Conn_01x02_MountingPin, U1 XIAO RA4M1, U2 TL074

Commit message: Updates to Unison board.
Parts:
- removed D1, D2, D3, D4: BAT43W-V, Diode_SMD:D_SOD-123, symbol Diode:BAT43W-V
- added D5: D1213A, CM_Chip_Packages:SOT-25, symbol CM_Device:DiodeArray_2ch
Connections:
- net +3V3: now also D5.5 (Vp)
- net GND_CH: now also D5.2 (Vn)
- net OSC2_VOL: now also D5.4 (CH2)
- net V-OCT: now also D5.3 (CH1)
