File: reference-designs/asmr-power-supply-reference/asmr-power-supply-reference-module-face-plate/asmr-power-supply-reference-module-face-plate.kicad_sch (KiCad schematic)
At the start: 0 parts

Commit message: Final Gerber tunings.
Other:
- title: Single Module Face Plate Reference Design -> Power Supply Module Face Plate
Changed lines of the file:
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@@
 	(paper "A4")
 	(title_block
-		(title "Single Module Face Plate Reference Design")
-		(date "2025-08-12")
+		(title "Power Supply Module Face Plate")
+		(date "2025-09-09")
 		(rev "A")
 		(company "by Circuit Monkey")
 		(comment 1 "ASMR :: Advanced Synth Module Rack")
-		(comment 2 "Face Plate for a AMSR Single Slot Module")
+		(comment 2 "Face Plate for AMSR Power Supply Module")
 	)
 	(wire
