File: modules/asmr-dreamland-proto-pad/asmr-dreamland-pcb/asmr-dreamland-pcb.kicad_sch (KiCad schematic)
At the start: 23 parts, among them J10 Conn_01x10, J11 Conn_01x10, J12 Conn_01x10, J13 Conn_01x10, J14 Conn_01x03, J15 Conn_01x03, J16 Conn_01x03, J17 Conn_01x03, J18 Conn_01x08, J2 Conn_01x06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

Commit message: Tune legend text.
Other:
- title: ASMR - Play Pen PCB Module -> DreamLand Proto Pad for ASMR
Changed lines of the file:
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@@
 	(paper "A4")
 	(title_block
-		(title "ASMR - Play Pen PCB Module")
-		(date "2025-08-20")
+		(title "DreamLand Proto Pad for ASMR")
+		(date "2025-09-09")
 		(rev "A")
 		(company "by Circuit Monkey")
-		(comment 1 "ASMR :: Advanced Synth Module Rack")
+		(comment 1 "for ASMR :: Advanced Synth Module Rack")
 		(comment 2 "Experimenters Playground PCB.")
 	)
