File: modules/asmr-dreamland-proto-pad/asmr-dreamland-pcb/asmr-dreamland-pcb.kicad_pcb (KiCad board)
At the start: 2 copper layers, 136 x 72 mm, 23 parts, among them J10 Conn_01x10, J11 Conn_01x10, J12 Conn_01x10, J13 Conn_01x10, J14 Conn_01x03, J15 Conn_01x03, J16 Conn_01x03, J17 Conn_01x03, J18 Conn_01x08, J2 Conn_01x06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

Commit message: Final tuning for DreamLand
Routing:
- added copper zone on B.Cu, net +15V
- added copper zone on F.Cu, net +15V
- added copper zone on B.Cu, net +18-24V
- added copper zone on F.Cu, net +18-24V
- added copper zone on B.Cu, net +5V
- added copper zone on F.Cu, net +5V
- added copper zone on B.Cu, net -15V
- added copper zone on F.Cu, net -15V
Other:
- board text added: "! Absolutely NOT PCI !"
- board text added: "DO NOT ATTEMPT TO USE IN A COMPUTER"
- board text added: "SMOKE, FIRE OR SMELLS MAY OCCUR"
