File: modules/asmr-dreamland-proto-pad/asmr-dreamland-face-plate/asmr-dreamland-face-plate.kicad_sch (KiCad schematic)
At the start: 0 parts

Commit message: Final tuning and gerber settings.
Other:
- title: DreamLand Module Face Plate -> DreamLand Prototyping Module Face Plate
Changed lines of the file:
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@@
 	(paper "A4")
 	(title_block
-		(title "DreamLand Module Face Plate")
-		(date "2025-08-12")
+		(title "DreamLand Prototyping Module Face Plate")
+		(date "2025-09-09")
 		(rev "A")
 		(company "by Circuit Monkey")
 		(comment 1 "for ASMR :: Advanced Synth Module Rack")
-		(comment 2 "Face Plate for DreamLand Module")
+		(comment 2 "Face Plate for DreamLand Prototyping Module")
 	)
 	(text "Notes:"
