File: modules/asmr-dreamland-proto-pad/asmr-dreamland-face-plate/asmr-dreamland-face-plate.kicad_pcb (KiCad board)
At the start: 2 copper layers, 40 x 159.6 mm, 0 parts

Commit message: Add JLC PCB serial tag to back silk.
Other:
- board text added: "JLCJLCJLCJLC"
Changed lines of the file:
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@@
+		)
+	)
+	(gr_text "JLCJLCJLCJLC"
+		(at 110 208 0)
+		(layer "B.SilkS")
+		(effects
+			(font
+				(size 1 1)
+				(thickness 0.15)
+			)
+			(justify mirror)
 		)
 	)
