File: reference-designs/asmr-power-supply-reference/asmr-power-supply-reference-module-pcb/asmr-power-supply-reference-module-pcb.kicad_pcb (KiCad board)
At the start: 2 copper layers, 136 x 72 mm, 74 parts, among them J2 USB_C_Receptacle_USB2.0_14P, J3 PWR-SW, Q1 DMP3036SFV, U1 HUSB238, U2 MP2328C, U3 MCP1365, U4 MP2328C

Commit message: Rev.B Notes and changes. Work in Progress.
Parts:
- R10, R12, R14: value 500K -> 499K
- R21: value 177K -> 178K
- U3: value MCP1365 -> MCP16365
Changed lines of the file:
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@@
 			)
 		)
-		(property "Value" "177K"
+		(property "Value" "178K"
 			(at 0 0.2 90)
 			(layer "F.Fab")
@@
 			)
 		)
-		(property "Value" "MCP1365"
+		(property "Value" "MCP16365"
 			(at 0.001384 2.105502 90)
 			(layer "F.Fab")
@@
 			)
 		)
-		(property "MPN" "MCP1365"
+		(property "MPN" "MCP16365"
 			(at 0 0 270)
 			(unlocked yes)
@@
 			)
 		)
-		(property "Value" "500K"
+		(property "Value" "499K"
 			(at 0 0.2 90)
 			(layer "F.Fab")
@@
 			)
 		)
-		(property "Value" "500K"
+		(property "Value" "499K"
 			(at 0 0.2 90)
 			(layer "F.Fab")
@@
 			)
 		)
-		(property "Value" "500K"
+		(property "Value" "499K"
 			(at 0 0.2 90)
 			(layer "F.Fab")
