File: modules/hagiwo-mod2/hagiwo-mod2.kicad_sch (KiCad schematic)
At the start: 72 parts, among them J1 JST-SH, J10 Conn_01x02_MountingPin, J2 JST-SH, J3 JST-SH, J4 Conn_01x02_MountingPin, J6 JST-SH, J7 Conn_01x02_MountingPin, J8 JST SH, 4P, VT, SMT, J9 Conn_01x02_MountingPin, U1 TL074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

Commit message: Add Rev.B notes and changes. Work in progress.
Parts:
- C11, C12, C5, C8, C9: value 1uF/50V -> 1uF/25V
- C18: value 0.01uF -> 1uF
- C6, C7: value 10uF/50V -> 10uF/25V
- R15: value 33.0K -> 45.0K
- R24: value 10K -> 100K
- R8: value 10K -> 33K
- RV2: MFR (none) -> Tayda; MPN (none) -> A-5538
- RV3: MFR (none) -> Tayda; MPN (none) -> A-5533
Other:
- note added: "Lengthen Package Pads"
- note added: "Maybe a GPIO FET controlled filter jumper here?"
- note added: "Strange place to put a TVS diode. Re-analyse where this might go. Move to TRS line?"
Changed lines of the file:
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@@
 	(title_block
 		(title "Hagiwo Mod2 Module")
-		(date "2025-09-08")
-		(rev "A")
+		(date "2025-09-30")
+		(rev "B")
 		(company "by Circuit Monkey")
 		(comment 1 "for ASMR - Advanced Synth Module Rack")
@@
 		)
 	)
+	(text "Lengthen\nPackage \nPads"
+		(exclude_from_sim no)
+		(at 136.906 78.486 0)
+		(effects
+			(font
+				(size 1.27 1.27)
+				(color 255 0 0 1)
+			)
+		)
+	)
 	(text "Pot 3"
 		(exclude_from_sim no)
@@
 		)
 	)
+	(text "Strange place to put a TVS diode.\nRe-analyse where this might go.\nMove to TRS line?"
+		(exclude_from_sim no)
+		(at 137.414 105.664 0)
+		(effects
+			(font
+				(size 1.27 1.27)
+				(color 255 0 0 1)
+			)
+		)
+	)
+	(text "Maybe a GPIO FET controlled filter jumper here?"
+		(exclude_from_sim no)
+		(at 236.22 159.512 0)
+		(effects
+			(font
+				(size 1.27 1.27)
+				(color 255 0 0 1)
+			)
+		)
+	)
 	(text "INPUT 1"
 		(exclude_from_sim no)
@@
 	)
 	(junction
-		(at 39.37 177.8)
-		(diameter 0)
-		(color 0 0 0 0)
-	)
-	(junction
 		(at 223.52 138.43)
 		(diameter 0)
@@
 	)
 	(junction
-		(at 43.18 121.92)
-		(diameter 0)
-		(color 0 0 0 0)
-	)
-	(junction
 		(at 275.59 81.28)
 		(diameter 0)
@@
 	(wire
 		(pts
-			(xy 41.91 121.92) (xy 43.18 121.92)
-		)
-		(stroke
-			(width 0)
-			(type default)
-		)
-	)
-	(wire
-		(pts
 			(xy 267.97 86.36) (xy 267.97 88.9)
 		)
@@
 	(wire
 		(pts
-			(xy 39.37 180.34) (xy 39.37 177.8)
-		)
-		(stroke
-			(width 0)
-			(type default)
-		)
-	)
-	(wire
-		(pts
 			(xy 223.52 138.43) (xy 223.52 140.97)
 		)
@@
 			)
 		)
-		(property "Value" "10uF/50V"
+		(property "Value" "10uF/25V"
 			(at 86.3587 166.5475 0)
 			(do_not_autoplace yes)
@@
 			)
 		)
-		(property "Value" "1uF/50V"
+		(property "Value" "1uF/25V"
 			(at 71.1187 165.2775 0)
 			(do_not_autoplace yes)
@@
 			)
 		)
-		(property "Value" "0.01uF"
+		(property "Value" "1uF"
 			(at 233.426 140.208 90)
 			(do_not_autoplace yes)
@@
 			)
 		)
-		(property "Value" "10uF/50V"
+		(property "Value" "10uF/25V"
 			(at 86.3587 158.9275 0)
 			(do_not_autoplace yes)
@@
 			)
 		)
+		(property "MPN" "A-5538"
+			(at 22.86 40.64 0)
+			(effects
+				(font
+					(size 1.27 1.27)
+				)
+				(hide yes)
+			)
+		)
+		(property "MFR" "Tayda"
+			(at 22.86 40.64 0)
+			(effects
+				(font
+					(size 1.27 1.27)
+				)
+				(hide yes)
+			)
+		)
 		(pin "2"
 		)
@@
 			)
 		)
-		(property "Value" "1uF/50V"
+		(property "Value" "1uF/25V"
 			(at 96.5187 158.9275 0)
 			(do_not_autoplace yes)
@@
 			)
 		)
-		(property "Value" "10K"
+		(property "Value" "100K"
 			(at 238.76 143.51 90)
 			(do_not_autoplace yes)
@@
 			)
 		)
+		(property "MPN" "A-5533"
+			(at 22.86 58.42 0)
+			(effects
+				(font
+					(size 1.27 1.27)
+				)
+				(hide yes)
+			)
+		)
+		(property "MFR" "Tayda"
+			(at 22.86 58.42 0)
+			(effects
+				(font
+					(size 1.27 1.27)
+				)
+				(hide yes)
+			)
+		)
 		(pin "2"
 		)
@@
 			)
 		)
-		(property "Value" "1uF/50V"
+		(property "Value" "1uF/25V"
 			(at 165.0987 176.7075 0)
 			(do_not_autoplace yes)
@@
 			)
 		)
-		(property "Value" "33.0K"
+		(property "Value" "45.0K"
 			(at 64.77 87.63 90)
 			(do_not_autoplace yes)
@@
 			)
 		)
-		(property "Value" "1uF/50V"
+		(property "Value" "1uF/25V"
 			(at 96.5187 166.5475 0)
 			(do_not_autoplace yes)
@@
 			)
 		)
-		(property "Value" "1uF/50V"
+		(property "Value" "1uF/25V"
 			(at 165.0987 186.8675 0)
 			(do_not_autoplace yes)
@@
 			)
 		)
-		(property "Value" "10K"
+		(property "Value" "33K"
 			(at 39.37 158.75 90)
 			(do_not_autoplace yes)

Commit message: Rev.B Tuning. Part values mostly.
Connections:
- net +3V3: now also RV1.3, RV2.3, RV3.3; no longer RV1.1, RV2.1, RV3.1
- net GND: now also RV1.1, RV2.1, RV3.1; no longer RV1.3, RV2.3, RV3.3
Changed lines of the file:
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@@
 		(lib_id "Device:R_Potentiometer_MountingPin")
 		(at 22.86 40.64 0)
+		(mirror x)
 		(unit 1)
 		(exclude_from_sim no)
@@
 		(dnp no)
 		(property "Reference" "RV2"
-			(at 25.908 37.338 0)
+			(at 25.4 37.084 0)
 			(do_not_autoplace yes)
 			(effects
@@
 		)
 		(property "Value" "100K"
-			(at 22.86 40.894 90)
+			(at 22.86 40.386 90)
 			(do_not_autoplace yes)
 			(effects
@@
 		(lib_id "Device:R_Potentiometer_MountingPin")
 		(at 22.86 21.59 0)
+		(mirror x)
 		(unit 1)
 		(exclude_from_sim no)
@@
 		(dnp no)
 		(property "Reference" "RV1"
-			(at 25.908 18.288 0)
+			(at 25.4 18.034 0)
 			(do_not_autoplace yes)
 			(effects
@@
 		)
 		(property "Value" "100K"
-			(at 22.86 21.844 90)
+			(at 22.86 21.336 90)
 			(do_not_autoplace yes)
 			(effects
@@
 		(lib_id "Device:R_Potentiometer_MountingPin")
 		(at 22.86 58.42 0)
+		(mirror x)
 		(unit 1)
 		(exclude_from_sim no)
@@
 		(dnp no)
 		(property "Reference" "RV3"
-			(at 25.908 55.118 0)
+			(at 25.4 54.864 0)
 			(do_not_autoplace yes)
 			(effects
@@
 		)
 		(property "Value" "10K"
-			(at 22.86 58.674 90)
-			(do_not_autoplace yes)
-			(effects
+			(at 22.86 58.166 90)
+			(do_not_autoplace yes)
+			(effects
